File: btn_ladder.kicad_sch (KiCad schematic)
At the start: 11 parts, among them SW2 TS24CA, SW4 TS24CA, SW5 TS24CA, SW6 TS24CA

Commit message: V1.0 or 4L final i hope
Parts:
- added R3: 10K, Resistor_SMD:R_0603_1608Metric, symbol Device:R_Small
- R38, R39: value 68K -> 10K
Connections:
- net ADCBTN_OUT: now also R3.2; no longer R33.2, SW4.4
- new net: R3.1, R33.2, SW4.4
Other:
- moved on the sheet: R31, R33, R34, R44, SW2, SW4, SW5, SW6
