File: electric_pass_baseboard.kicad_pcb (KiCad board)
At the start: 2 copper layers, 50 x 100 mm, 146 parts, among them J1 USB_C_Receptacle_USB2.0_16P, J2 Conn_02x05_Counter_Clockwise, J3 Conn_02x05_Counter_Clockwise, Q1 AO3401A, Q2 AO3401A, SW1 TS24CA, SW2 TS24CA, SW4 TS24CA, SW5 TS24CA, SW6 TS24CA, SW9 TS24CA, U1 TP4056-42-ESOP8, U10 ZX-SH1.0-2PWT, U2 EA3036C, U3 F1C200S, U4 3寸液晶屏TFT 全新无定义资料, U5 ST7701 IPS, U6 W25N01GVZEIG_C907680, U8 GEK100-XX, U9 STI9287C, Y1 24Mhz 12pF

Commit message: 0.5.1 4 layer.
Parts:
- moved U8 0.06 mm to (134.8, 127.8)
Connections:
- U8 pad 1: VBAT -> Net-(U8-KEY)
- U8 pad 3: Net-(U8-KEY) -> /power/PWR_SHUTDOWN
- U8 pad 4: /power/PWR_SHUTDOWN -> Net-(Q2-G)
- U8 pad 5: Net-(Q2-G) -> unconnected-(U8-OUTH-Pad5)
- U8 pad 6: unconnected-(U8-OUTH-Pad6) -> VBAT
Routing:
- net VBUS: track 54.2 -> 60.0 mm
- net /power/PWR_SHUTDOWN: track 51.2 -> 56.3 mm, vias 2 -> 4
- net GND: track 155.6 -> 152.6 mm
- net /VBAT_SENSE: track 58.9 -> 60.3 mm
- net Net-(Q2-G): track 7.98 -> 9.16 mm
- net /ADC: track 45.4 -> 46.4 mm
- net /USB_DN: track 46.0 -> 46.9 mm
- net VBAT: track 54.4 -> 55.3 mm, vias 4 -> 5
- net /UART1_RX: track 43.8 -> 44.5 mm
- net Net-(U8-KEY): track 7.49 -> 8.13 mm
- net /PE3: track 62.0 -> 62.6 mm
- net /USB_DP: track 46.4 -> 46.9 mm
- added copper zone on In1.Cu, net GND
- added copper zone on In2.Cu, net GND
Other:
- copper layers 2 -> 4
- board text added: "Electronic Authorization Terminal 电子通行证终端 Model/型号: EPA-V051 Power/电源: 5V1A ACC ID: 1238fe1 LMIIT ID: 7355613 拉特兰机械制造总局受托制造"
- board text added: "Rhodes Island Electric Pass V0.5.1 4L Ver."
- board text removed: "Electronic Authorization Terminal 电子通行证终端 Model/型号: EPA-V04 Power/电源: 5V1A ACC ID: 3279ade LMIIT ID: 7355611 拉特兰机械制造总局受托制造"
- board text removed: "Rhodes Island Electric Pass V0.5"

Commit message: V1.0 or 4L final i hope
Parts:
- removed F1: Fuse, Fuse:Fuse_0805_2012Metric
- added C38: 10uF, Capacitor_SMD:C_0603_1608Metric, F.Cu at (144.8, 120.1)
- added D6: 1N5819WS, shirogane:D_SOD-323, F.Cu at (133.8, 96.7)
- added D7: ESD5Z3V3, Diode_SMD:D_SOD-523, F.Cu at (150.6, 135.1)
- added D8: ESD5Z3V3, Diode_SMD:D_SOD-523, F.Cu at (147.8, 135.1)
- added R3: 10K, Resistor_SMD:R_0603_1608Metric, F.Cu at (133.4, 88.6)
- added R4: 10K, Resistor_SMD:R_0603_1608Metric, F.Cu at (137.9, 127.9)
- added R43: 2K, Resistor_SMD:R_0603_1608Metric, F.Cu at (141.3, 123.7)
- added R45: 2K, Resistor_SMD:R_0603_1608Metric, F.Cu at (141.3, 125.2)
- added U7: PW1515, Package_TO_SOT_SMD:SOT-23-5, F.Cu at (145.1, 137.5)
- D2, D5: footprint Diode_SMD:D_SOD-323 -> shirogane:D_SOD-323
- FID1, FID2, FID4: footprint Fiducial:Fiducial_1mm_Mask3mm -> shirogane:Fiducial_1mm_Mask3mm
- R38, R39: value 68K -> 10K
- moved C37 19.0 mm to (144.0, 106.6), turned to 0 degrees
- moved U6 13.1 mm to (136.3, 103.3), turned to -90 degrees
- moved TP11 11.0 mm to (142.3, 119.1)
- moved R28 9.86 mm to (161.8, 81.9), turned to -90 degrees
- moved R2 8.69 mm to (152.7, 136.6), turned to 0 degrees
- moved TP3 8.63 mm to (168.1, 110.7)
- moved Q1 8.62 mm to (144.8, 124.7), turned to 90 degrees
- moved D2 8.60 mm to (144.7, 121.8), turned to 180 degrees
- moved R7 8.41 mm to (163.3, 81.9), turned to -90 degrees
- moved R5 8.30 mm to (144.0, 109.2)
- moved R6 8.12 mm to (144.1, 110.9)
- moved R1 7.51 mm to (152.9, 138.5)
- moved R8 6.89 mm to (144.0, 114.0)
- moved R35 6.84 mm to (144.1, 115.6)
- moved R36 6.76 mm to (144.0, 117.2)
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Connections:
- net Net-(F1-Pad1) renamed /VBUS_IN
- C47 pad 1: VBAT -> Net-(D2-K)
- R31 pad 1: /adc_periph/ADCBTN_OUT -> /PWR_BTN
- R33 pad 2: /adc_periph/ADCBTN_OUT -> Net-(R3-Pad1)
- SW4 pad 4: /adc_periph/ADCBTN_OUT -> Net-(R3-Pad1)
- U3 pad 79: /adc_periph/ADCBTN_OUT -> /PWR_BTN
- U8 pad 6: VBAT -> Net-(D2-K)
- Y1 pad 2: unconnected-(Y1-Pad2) -> GND
- Y1 pad 4: unconnected-(Y1-Pad4) -> GND
Routing:
- net VBAT_OUT: track 129.3 -> 60.0 mm, vias 15 -> 29
- net /adc_periph/ADCBTN_OUT: track 50.6 -> 0.00 mm, vias 2 -> 0
- net Net-(D6-K): track 8.13 -> 53.7 mm
- net /PWR_BTN: track 0.00 -> 36.8 mm, vias 0 -> 2
- net /screen/SCREEN_BL_CTRL: track 53.1 -> 22.9 mm
- net /soc_f1c/SDIO_CLK: track 31.6 -> 53.3 mm
- net +3.3V: track 282.9 -> 304.4 mm, vias 24 -> 53
- net /UART0_RX: track 47.7 -> 66.9 mm, vias 0 -> 2
- net Net-(U7-IADJ): track 0.00 -> 18.3 mm
- net Net-(R3-Pad1): track 0.00 -> 17.9 mm
- net /PE5: track 48.5 -> 65.9 mm, vias 0 -> 2
- net /VBUS_IN: track 9.13 -> 25.3 mm
- net /SPI1_CS: track 50.7 -> 66.7 mm, vias 0 -> 2
- net /soc_f1c/SDIO_D2: track 39.5 -> 55.0 mm
- net /soc_f1c/SDIO_D3: track 39.8 -> 55.0 mm
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- added copper zone on In2.Cu, net +1V2
- added copper zone on In2.Cu, net +2V5
- added copper zone on In2.Cu, net +3.3V
- added copper zone on F.Cu, net Net-(D2-K)
- added copper zone on In2.Cu, net Net-(D2-K)
- added copper zone on In2.Cu, net VBAT_OUT
- added copper zone on F.Cu, net VBUS
- added copper zone on In2.Cu, net VBUS
- removed copper zone on B.Cu, net +1V2
- removed copper zone on B.Cu, net +2V5
- removed copper zone on B.Cu, net +3.3V
- removed copper zone on B.Cu, net VBAT_OUT
Other:
- board text added: "*1->"
- board text added: "*1:PA1脚功能 安装：采集电量 不安装：外部IO *2:老五屏贴装 *3:常规屏贴装 *4:默认开背光 *5:默认关背光"
- board text added: "*2->"
- board text added: "*4->"
- board text added: "*5->"
- board text added: "<-*2"
- board text added: "<-*3"
- board text added: "Bat.CHG"
- board text added: "DC-DC"
- board text added: "DFM： 1. LRADC过孔越少越好。且加大线宽，加大过孔， 防止孔电阻不合格，导致按钮检测出错。 2. USB保证完整地平面，保证完好的回流路径。给完全的一层地"
- board text added: "Electronic Authorization Terminal 电子通行证终端 Model/型号: EPA-4L-V1 Power/电源: 5V1A ACC ID: sad3e4 LMIIT ID: 7355614 拉特兰机械制造总局受托制造"
- board text added: "F1C200S"
- board text added: "JLC04101H-3313 90 共面差分阻抗（外层） W:5.5 差分间距：6 到铜距离：8"
- board text added: "NAND"
- board text added: "PRTS Infomation"
- board text added: "Rhodes Island Electronic Pass 4L V1.0"
- board text added: "Screen"
- board text added: "充电 充满 ↓ ↓"
- board text added: "看不懂就贴*1*4, *2*3根据你的屏选"
- board text added: "运行中"
- board text removed: "Electronic Authorization Terminal 电子通行证终端 Model/型号: EPA-V051 Power/电源: 5V1A ACC ID: 1238fe1 LMIIT ID: 7355613 拉特兰机械制造总局受托制造"
- board text removed: "Rhodes Island Electric Pass V0.5.1 4L Ver."
