File: electric_pass_baseboard.kicad_sch (KiCad schematic)
At the start: 17 parts, among them J1 USB_C_Receptacle_USB2.0_16P, J2 Conn_02x05_Counter_Clockwise, J3 Conn_02x05_Counter_Clockwise

Commit message: 0.5.1 4 layer.
Other:
- note added: "特别感谢：（不分先后）和光、薄云、烟雨、WXNA、 土豆、星语Studio、爱莉希雅、所有复刻群友的支持！"
Changed lines of the file:
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@@
 		(comment 1 "V0.3 添加屏幕兼容接口，添加SD卡槽，优化布线")
 		(comment 2 "V0.3.1 BUG修复")
-		(comment 3 "土豆、星语Studio、爱莉希雅、所有复刻群友的支持！")
-		(comment 4 "V0.3.2 生产优化。特别感谢：（不分先后）和光、薄云、烟雨、WXNA、")
+		(comment 3 "V0.3.2（V0.4） 生产优化。")
+		(comment 4 "V0.5 实现按键开关机、低电量关机、拉出i2s")
 	)
 	(text "贴10R省一种料"
@@
 				(size 1.27 1.27)
 			)
+		)
+	)
+	(text "特别感谢：（不分先后）和光、薄云、烟雨、WXNA、\n土豆、星语Studio、爱莉希雅、所有复刻群友的支持！\n"
+		(exclude_from_sim no)
+		(at 213.614 149.352 0)
+		(effects
+			(font
+				(size 1.27 1.27)
+			)
+			(justify left)
 		)
 	)
@@
 		)
 	)
+	(netclass_flag ""
+		(length 2.54)
+		(shape round)
+		(at 87.63 91.44 0)
+		(fields_autoplaced yes)
+		(effects
+			(font
+				(size 1.27 1.27)
+			)
+			(justify left bottom)
+		)
+		(property "Netclass" "USB"
+			(at 88.3285 88.9 0)
+			(effects
+				(font
+					(size 1.27 1.27)
+				)
+				(justify left)
+			)
+		)
+		(property "Component Class" ""
+			(at -60.96 7.62 0)
+			(effects
+				(font
+					(size 1.27 1.27)
+					(italic yes)
+				)
+			)
+		)
+	)
+	(netclass_flag ""
+		(length 2.54)
+		(shape round)
+		(at 83.82 86.36 0)
+		(fields_autoplaced yes)
+		(effects
+			(font
+				(size 1.27 1.27)
+			)
+			(justify left bottom)
+		)
+		(property "Netclass" "USB"
+			(at 84.5185 83.82 0)
+			(effects
+				(font
+					(size 1.27 1.27)
+				)
+				(justify left)
+			)
+		)
+		(property "Component Class" ""
+			(at -64.77 2.54 0)
+			(effects
+				(font
+					(size 1.27 1.27)
+					(italic yes)
+				)
+			)
+		)
+	)

Commit message: V1.0 or 4L final i hope
Parts:
- removed F1: Fuse, Fuse:Fuse_0805_2012Metric, symbol Device:Fuse
- added C38: 10uF, Capacitor_SMD:C_0603_1608Metric, symbol Device:C_Small
- added D7, D8: ESD5Z3V3, Diode_SMD:D_SOD-523, symbol Diode:ESD5Zxx
- added R43, R45: 2K, Resistor_SMD:R_0603_1608Metric, symbol Device:R_Small
- added U7: PW1515, Package_TO_SOT_SMD:SOT-23-5, symbol shirogane:PW1515
- TP10, TP4, TP5, TP7, TP8, TP9: footprint TestPoint:TestPoint_Pad_D1.5mm -> TestPoint:TestPoint_Pad_D1.0mm
Connections:
- net GND: now also C38.2, D7.2 (A), D8.2 (A), R43.1, R45.1, U7.2 (GND)
- net USB_DN: now also D8.1 (K)
- net USB_DP: now also D7.1 (K)
- net VBUS: now also C38.1, U7.1 (VOUT)
- net VBUS_IN: now reaches J1.A4 (VBUS), J1.A9 (VBUS), J1.B4 (VBUS), J1.B9 (VBUS)
- net VBUS_IN: now also U7.5 (VIN)
- new net: R43.2, R45.2, U7.3 (IADJ)
- no-connect marks 2 -> 3
Other:
- sheet adc_periph ports: added PWR_BTN; removed none
- sheet power ports: added PWR_BTN; removed none
- note added: "*1：ADC1用于电池采样功能选择 若拆焊R40 ，则ADC可用于外部IO，但会失去电池电量检测功能"
- note added: "特别感谢：（不分先后）和光、薄云、烟雨、WXNA、西南季风、“你说得对” 土豆、星语Studio、爱莉希雅、所有复刻群友的支持！"
- note added: "过压/过流保护 我麻了啊，怎么快冲还会误触发的 感谢：西南季风大哥！ I_OCP = 600/1000 = 0.6A"
- note removed: "特别感谢：（不分先后）和光、薄云、烟雨、WXNA、 土豆、星语Studio、爱莉希雅、所有复刻群友的支持！"
- note removed: "贴10R省一种料"
