File: power.kicad_sch (KiCad schematic)
At the start: 52 parts, among them Q1 AO3401A, Q2 AO3401A, SW1 TS24CA, U1 TP4056-42-ESOP8, U10 ZX-SH1.0-2PWT, U2 EA3036C, U8 GEK100-XX

Commit message: 0.5.1 4 layer.
Connections:
- net PWR_SHUTDOWN: now also U8.3 (RST); no longer U8.4 (RST)
- net VBAT: now also U8.6 (VDD); no longer U8.1 (VDD)
- net at SW1.4: now also U8.1 (KEY); no longer U8.3 (KEY)
- net at Q2.1 (G): now also U8.4 (OUTL); no longer U8.5 (OUTL)
Other:
- note added: "按键开关机（低压保护也靠这个切断） 感谢群友：“你说得对”、**星语Studio** 、土豆、量子！"
- note removed: "按键开关机（低压保护也靠这个切断） 感谢群友：“你说得对”、星语Studio、土豆、量子！"
Changed lines of the file:
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@@
 		(comment 1 "V0.3 添加屏幕兼容接口，添加SD卡槽，优化布线")
 		(comment 2 "V0.3.1 BUG修复")
-		(comment 3 "土豆、星语Studio、爱莉希雅、所有复刻群友的支持！")
-		(comment 4 "V0.3.2 生产优化。特别感谢：（不分先后）和光、薄云、烟雨、WXNA、")
+		(comment 3 "V0.3.2（V0.4） 生产优化。")
+		(comment 4 "V0.5 实现按键开关机、低电量关机、拉出i2s")
 	)
-	(text "按键开关机（低压保护也靠这个切断）\n感谢群友：“你说得对”、星语Studio、土豆、量子！"
+	(text "按键开关机（低压保护也靠这个切断）\n感谢群友：“你说得对”、**星语Studio**\n、土豆、量子！"
 		(exclude_from_sim no)
-		(at 82.804 108.966 0)
+		(at 83.058 103.124 0)
 		(effects
 			(font

Commit message: V1.0 or 4L final i hope
Parts:
- added D6: 1N5819WS, shirogane:D_SOD-323, symbol Diode:1N5819WS
- added R4: 10K, Resistor_SMD:R_0603_1608Metric, symbol Device:R_Small
- D2: footprint Diode_SMD:D_SOD-323 -> shirogane:D_SOD-323
Connections:
- net VBAT: no longer C47.1, U8.6 (VDD)
- net at SW1.4, U8.1 (KEY): now also D6.1 (K), R4.1
- net at D2.1 (K), Q1.2 (S), Q2.2 (S): now also C47.1, U8.6 (VDD), R4.2
- new net PWR_BTN: D6.2 (A)
Other:
- moved on the sheet: C47, D4, R12, SW1
