File: screen.kicad_sch (KiCad schematic)
At the start: 17 parts, among them U4 3寸液晶屏TFT 全新无定义资料, U5 ST7701 IPS, U9 STI9287C

Commit message: V1.0 or 4L final i hope
Parts:
- D5: footprint Diode_SMD:D_SOD-323 -> shirogane:D_SOD-323
- R28: 特殊说明 (none) -> 贴了默认开背光
- R7: 特殊说明 不贴装 -> 贴了默认关背光
- U5: footprint Connector_FFC-FPC:Hirose_FH12-40S-0.5SH_1x40-1MP_P0.50mm_Horizontal -> shirogane:FPC-SMD_40P-P0.50_HC-FPC-0.5-40P-CSH20
Other:
- note added: "*4/*5:开机默认背光状态 贴R28: 默认开背光 贴R7：默认关背光 手动复刻建议贴R28 调试结束后贴R7 批量直接R7+QC"
- note added: "Alt.BOM:SY7200A"
Changed lines of the file:
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@@
 		(comment 4 "V0.5 实现按键开关机、低电量关机、拉出i2s")
 	)
+	(text "*4/*5:开机默认背光状态\n贴R28: 默认开背光\n贴R7：默认关背光\n\n手动复刻建议贴R28 调试结束后贴R7\n批量直接R7+QC"
+		(exclude_from_sim no)
+		(at 194.056 137.668 0)
+		(effects
+			(font
+				(size 1.27 1.27)
+			)
+		)
+	)
 	(text "RSense = 0.2 / I_LED \n       = 10 Ohm"
 		(exclude_from_sim no)
@@
 	(text "EN Dimming with wide PWM Frequency\nRange: 1kHz to 200kHz\n"
 		(exclude_from_sim no)
-		(at 225.298 139.446 0)
+		(at 234.188 136.652 0)
 		(effects
 			(font
@@
 		(exclude_from_sim no)
 		(at 269.24 102.616 0)
+		(effects
+			(font
+				(size 1.27 1.27)
+			)
+		)
+	)
+	(text "Alt.BOM:SY7200A"
+		(exclude_from_sim no)
+		(at 225.044 122.682 0)
 		(effects
 			(font
@@
 			)
 		)
-		(property "Footprint" "Connector_FFC-FPC:Hirose_FH12-40S-0.5SH_1x40-1MP_P0.50mm_Horizontal"
+		(property "Footprint" "shirogane:FPC-SMD_40P-P0.50_HC-FPC-0.5-40P-CSH20"
 			(at 134.366 157.988 0)
 			(effects
@@
 			)
 		)
-		(property "Footprint" "Diode_SMD:D_SOD-323"
+		(property "Footprint" "shirogane:D_SOD-323"
 			(at 243.84 93.345 0)
 			(effects
@@
 			)
 		)
+		(property "特殊说明" "贴了默认开背光"
+			(at 200.66 119.38 90)
+			(effects
+				(font
+					(size 1.27 1.27)
+				)
+				(hide yes)
+			)
+		)
 		(pin "1"
 		)
@@
 			)
 		)
-		(property "特殊说明" "不贴装"
+		(property "特殊说明" "贴了默认关背光"
 			(at 200.66 127 90)
 			(effects
